File: KiCad/bbc-keyboard/bbc-keyboard.kicad_pcb (KiCad board)
At the start: 2 copper layers, 75 parts, among them SW1 escape, SW10 W, SW11 2, SW12 A, SW13 S, SW14 Z, SW15 f2, SW16 4, SW17 E, SW18 D, SW19 X, SW2 Q, SW20 C, SW21 space, SW22 f3, SW23 5, SW24 T, SW25 R, SW26 F, SW27 G, SW28 V, SW29 f5, SW3 F0, SW30 F4, SW31 7, SW32 6, SW33 Y, SW34 H, SW35 B, SW36 f6, SW37 8, SW38 9, SW39 U, SW4 1, SW40 J, SW41 N, SW42 M, SW43 f8, SW44 f7, SW45 I, SW46 O, SW47 K, SW48 L, SW49 <,, SW5 caps lk, SW50 f9, SW51 =-, SW52 0, SW53 P, SW54 @, SW55 ;+, SW56 >., SW57 \|, SW58 ~^, SW59 _£, SW6 shift lk, SW60 {[, SW61 *:, SW62 }], SW63 ?/, SW64 right, SW65 left, SW66 down, SW67 up, SW68 return, SW69 delete, SW7 tab, SW70 copy, SW71 shift, SW72 shift, SW73 ctrl, SW75 break, SW8 f1, SW9 3

Commit message: Added - original outlines
Parts:
- moved RP1 37.0 mm to (218.4, 101.6)
- moved SW1 37.0 mm to (76.2, 139.7)
- moved SW13 37.0 mm to (128.6, 177.8)
- moved SW16 37.0 mm to (152.4, 139.7)
- moved SW19 37.0 mm to (138.1, 196.8)
- moved SW2 37.0 mm to (104.8, 158.8)
- moved SW22 37.0 mm to (176.2, 120.7)
- moved SW25 37.0 mm to (161.9, 158.8)
- moved SW26 37.0 mm to (166.7, 177.8)
- moved SW27 37.0 mm to (185.7, 177.8)
- moved SW28 37.0 mm to (176.2, 196.8)
- moved SW29 37.0 mm to (214.3, 120.7)
- moved SW31 37.0 mm to (209.6, 139.7)
- moved SW32 37.0 mm to (190.5, 139.7)
- moved SW33 37.0 mm to (200.0, 158.8)
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
Commit message: LEDs
Parts:
- added LD1: SHIFT, LED_THT:LED_D5.0mm, F.Cu at (113.3, 224.8)
- added LD2: CAPS, LED_THT:LED_D5.0mm, F.Cu at (93.0, 224.8)
- added LD3: CAS, LED_THT:LED_D5.0mm, F.Cu at (72.7, 224.8)
Other:
- board outline added: 337.8 x 137.2 mm
Changed lines of the file:
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@@
   (net 22 "GND")
   (net 23 "/~{RST}")
+  (net 24 "Net-(LD1-Pad1)")
+  (net 25 "Net-(LD2-Pad1)")
+  (net 26 "Net-(LD3-Pad1)")
   (footprint "Switch_Keyboard_Cherry_MX:SW_Cherry_MX_PCB_1.00u" (layer "F.Cu")
     (at 104.775 158.75)
@@
     )
   )
+  (footprint "LED_THT:LED_D5.0mm" (layer "F.Cu")
+    (at 72.7025 224.79)
+    (descr "LED, diameter 5.0mm, 2 pins, http://cdn-reichelt.de/documents/datenblatt/A500/LL-504BC2E-009.pdf")
+    (tags "LED diameter 5.0mm 2 pins")
+    (property "Sheetfile" "bbc-keyboard.kicad_sch")
+    (property "Sheetname" "")
+    (attr through_hole)
+    (fp_text reference "LD3" (at 1.27 -3.96) (layer "F.SilkS")
+      (effects (font (size 1 1) (thickness 0.15)))
+    )
+    (fp_text value "CAS" (at 1.27 3.96) (layer "F.Fab")
+      (effects (font (size 1 1) (thickness 0.15)))
+    )
+    (fp_text user "${REFERENCE}" (at 1.25 0) (layer "F.Fab")
+      (effects (font (size 0.8 0.8) (thickness 0.2)))
+    )
+    (fp_line (start -1.29 -1.545) (end -1.29 1.545) (layer "F.SilkS") (width 0.12))
+    (fp_arc (start -1.29 -1.54483) (mid 2.072002 -2.880433) (end 4.26 0.000462) (layer "F.SilkS") (width 0.12))
+    (fp_arc (start 4.26 -0.000462) (mid 2.072002 2.880433) (end -1.29 1.54483) (layer "F.SilkS") (width 0.12))
+    (fp_circle (center 1.27 0) (end 3.77 0) (layer "F.SilkS") (width 0.12) (fill none))
+    (fp_line (start -1.95 3.25) (end 4.5 3.25) (layer "F.CrtYd") (width 0.05))
+    (fp_line (start 4.5 -3.25) (end -1.95 -3.25) (layer "F.CrtYd") (width 0.05))
+    (fp_line (start 4.5 3.25) (end 4.5 -3.25) (layer "F.CrtYd") (width 0.05))
+    (fp_line (start -1.95 -3.25) (end -1.95 3.25) (layer "F.CrtYd") (width 0.05))
+    (fp_line (start -1.23 -1.469694) (end -1.23 1.469694) (layer "F.Fab") (width 0.1))
+    (fp_arc (start -1.23 -1.469694) (mid 4.17 0.000016) (end -1.230016 1.469666) (layer "F.Fab") (width 0.1))
+    (fp_circle (center 1.27 0) (end 3.77 0) (layer "F.Fab") (width 0.1) (fill none))
+    (pad "1" thru_hole rect (at 0 0) (size 1.8 1.8) (drill 0.9) (layers *.Cu *.Mask)
+      (net 26 "Net-(LD3-Pad1)") (pinfunction "K") (pintype "passive"))
+    (pad "2" thru_hole circle (at 2.54 0) (size 1.8 1.8) (drill 0.9) (layers *.Cu *.Mask)
+      (net 1 "VCC") (pinfunction "A") (pintype "passive"))
+    (model "${KICAD6_3DMODEL_DIR}/LED_THT.3dshapes/LED_D5.0mm.wrl"
+      (offset (xyz 0 0 0))
+      (scale (xyz 1 1 1))
+      (rotate (xyz 0 0 0))
+    )
+  )
   (footprint "Switch_Keyboard_Cherry_MX:SW_Cherry_MX_PCB_1.00u" (layer "F.Cu")
     (at 76.2 139.7)
@@
     )
   )
+  (footprint "LED_THT:LED_D5.0mm" (layer "F.Cu")
+    (at 93.0225 224.79)
+    (descr "LED, diameter 5.0mm, 2 pins, http://cdn-reichelt.de/documents/datenblatt/A500/LL-504BC2E-009.pdf")
+    (tags "LED diameter 5.0mm 2 pins")
+    (property "Sheetfile" "bbc-keyboard.kicad_sch")
+    (property "Sheetname" "")
+    (attr through_hole)
+    (fp_text reference "LD2" (at 1.27 -3.96) (layer "F.SilkS")
+      (effects (font (size 1 1) (thickness 0.15)))
+    )
+    (fp_text value "CAPS" (at 1.27 3.96) (layer "F.Fab")
+      (effects (font (size 1 1) (thickness 0.15)))
+    )
+    (fp_text user "${REFERENCE}" (at 1.25 0) (layer "F.Fab")
+      (effects (font (size 0.8 0.8) (thickness 0.2)))
+    )
+    (fp_line (start -1.29 -1.545) (end -1.29 1.545) (layer "F.SilkS") (width 0.12))
+    (fp_arc (start 4.26 -0.000462) (mid 2.072002 2.880433) (end -1.29 1.54483) (layer "F.SilkS") (width 0.12))
+    (fp_arc (start -1.29 -1.54483) (mid 2.072002 -2.880433) (end 4.26 0.000462) (layer "F.SilkS") (width 0.12))
+    (fp_circle (center 1.27 0) (end 3.77 0) (layer "F.SilkS") (width 0.12) (fill none))
+    (fp_line (start 4.5 -3.25) (end -1.95 -3.25) (layer "F.CrtYd") (width 0.05))
+    (fp_line (start -1.95 -3.25) (end -1.95 3.25) (layer "F.CrtYd") (width 0.05))
+    (fp_line (start 4.5 3.25) (end 4.5 -3.25) (layer "F.CrtYd") (width 0.05))
+    (fp_line (start -1.95 3.25) (end 4.5 3.25) (layer "F.CrtYd") (width 0.05))
+    (fp_line (start -1.23 -1.469694) (end -1.23 1.469694) (layer "F.Fab") (width 0.1))
+    (fp_arc (start -1.23 -1.469694) (mid 4.17 0.000016) (end -1.230016 1.469666) (layer "F.Fab") (width 0.1))
+    (fp_circle (center 1.27 0) (end 3.77 0) (layer "F.Fab") (width 0.1) (fill none))
+    (pad "1" thru_hole rect (at 0 0) (size 1.8 1.8) (drill 0.9) (layers *.Cu *.Mask)
+      (net 25 "Net-(LD2-Pad1)") (pinfunction "K") (pintype "passive"))
+    (pad "2" thru_hole circle (at 2.54 0) (size 1.8 1.8) (drill 0.9) (layers *.Cu *.Mask)
+      (net 1 "VCC") (pinfunction "A") (pintype "passive"))
+    (model "${KICAD6_3DMODEL_DIR}/LED_THT.3dshapes/LED_D5.0mm.wrl"
+      (offset (xyz 0 0 0))
+      (scale (xyz 1 1 1))
+      (rotate (xyz 0 0 0))
+    )
+  )
   (footprint "Switch_Keyboard_Cherry_MX:SW_Cherry_MX_PCB_1.00u" (layer "F.Cu")
     (at 371.475 158.75)
@@
     )
   )
+  (footprint "LED_THT:LED_D5.0mm" (layer "F.Cu")
+    (at 113.3425 224.79)
+    (descr "LED, diameter 5.0mm, 2 pins, http://cdn-reichelt.de/documents/datenblatt/A500/LL-504BC2E-009.pdf")
+    (tags "LED diameter 5.0mm 2 pins")
+    (property "Sheetfile" "bbc-keyboard.kicad_sch")
+    (property "Sheetname" "")
+    (attr through_hole)
+    (fp_text reference "LD1" (at 1.27 -3.96) (layer "F.SilkS")
+      (effects (font (size 1 1) (thickness 0.15)))
+    )
+    (fp_text value "SHIFT" (at 1.27 3.96) (layer "F.Fab")
+      (effects (font (size 1 1) (thickness 0.15)))
+    )
+    (fp_text user "${REFERENCE}" (at 1.25 0) (layer "F.Fab")
+      (effects (font (size 0.8 0.8) (thickness 0.2)))
+    )
+    (fp_line (start -1.29 -1.545) (end -1.29 1.545) (layer "F.SilkS") (width 0.12))
+    (fp_arc (start 4.26 -0.000462) (mid 2.072002 2.880433) (end -1.29 1.54483) (layer "F.SilkS") (width 0.12))
+    (fp_arc (start -1.29 -1.54483) (mid 2.072002 -2.880433) (end 4.26 0.000462) (layer "F.SilkS") (width 0.12))
+    (fp_circle (center 1.27 0) (end 3.77 0) (layer "F.SilkS") (width 0.12) (fill none))
+    (fp_line (start 4.5 -3.25) (end -1.95 -3.25) (layer "F.CrtYd") (width 0.05))
+    (fp_line (start 4.5 3.25) (end 4.5 -3.25) (layer "F.CrtYd") (width 0.05))
+    (fp_line (start -1.95 3.25) (end 4.5 3.25) (layer "F.CrtYd") (width 0.05))
+    (fp_line (start -1.95 -3.25) (end -1.95 3.25) (layer "F.CrtYd") (width 0.05))
+    (fp_line (start -1.23 -1.469694) (end -1.23 1.469694) (layer "F.Fab") (width 0.1))
+    (fp_arc (start -1.23 -1.469694) (mid 4.17 0.000016) (end -1.230016 1.469666) (layer "F.Fab") (width 0.1))
+    (fp_circle (center 1.27 0) (end 3.77 0) (layer "F.Fab") (width 0.1) (fill none))
+    (pad "1" thru_hole rect (at 0 0) (size 1.8 1.8) (drill 0.9) (layers *.Cu *.Mask)
+      (net 24 "Net-(LD1-Pad1)") (pinfunction "K") (pintype "passive"))
+    (pad "2" thru_hole circle (at 2.54 0) (size 1.8 1.8) (drill 0.9) (layers *.Cu *.Mask)
+      (net 1 "VCC") (pinfunction "A") (pintype "passive"))
+    (model "${KICAD6_3DMODEL_DIR}/LED_THT.3dshapes/LED_D5.0mm.wrl"
+      (offset (xyz 0 0 0))
+      (scale (xyz 1 1 1))
+      (rotate (xyz 0 0 0))
+    )
+  )
   (footprint "Switch_Keyboard_Cherry_MX:SW_Cherry_MX_PCB_1.00u" (layer "F.Cu")
     (at 252.4125 120.65)
@@
   (gr_line (start 312.7375 232.41) (end 58.7375 232.41) (layer "Dwgs.User") (width 0.15))
   (gr_line (start 368.6175 213.36) (end 312.7375 213.36) (layer "Dwgs.User") (width 0.15))
+  (gr_circle (center 73.9775 224.79) (end 77.1525 224.79) (layer "Dwgs.User") (width 0.15) (fill none))
   (gr_line (start 58.7375 127) (end 96.8375 127) (layer "Dwgs.User") (width 0.15))
   (gr_line (start 96.8375 127) (end 96.8375 107.95) (layer "Dwgs.User") (width 0.15))
@@
   (gr_line (start 58.7375 232.41) (end 15.5575 232.41) (layer "Dwgs.User") (width 0.15))
   (gr_line (start 20.6375 201.93) (end 20.6375 199.39) (layer "Dwgs.User") (width 0.15))
+  (gr_circle (center 94.2975 224.79) (end 97.4725 224.79) (layer "Dwgs.User") (width 0.15) (fill none))
   (gr_line (start 312.7375 213.36) (end 312.7375 232.41) (layer "Dwgs.User") (width 0.15))
   (gr_line (start 391.4775 201.93) (end 391.4775 199.39) (layer "Dwgs.User") (width 0.15))
@@
   (gr_circle (center 33.3375 200.66) (end 39.6875 200.66) (layer "Dwgs.User") (width 0.15) (fill none))
   (gr_circle (center 378.7775 200.66) (end 385.1275 200.66) (layer "Dwgs.User") (width 0.15) (fill none))
+  (gr_circle (center 20.6375 158.75) (end 23.1775 158.75) (layer "Dwgs.User") (width 0.15) (fill none))
+  (gr_circle (center 390.2075 158.75) (end 392.7475 158.75) (layer "Dwgs.User") (width 0.15) (fill none))
   (gr_line (start 383.8575 107.95) (end 383.8575 191.77) (layer "Dwgs.User") (width 0.15))
+  (gr_circle (center 114.6175 224.79) (end 117.7925 224.79) (layer "Dwgs.User") (width 0.15) (fill none))
   (gr_line (start 15.5575 232.41) (end 15.5575 82.55) (layer "Dwgs.User") (width 0.15))
   (gr_line (start 58.7375 232.41) (end 58.7375 127) (layer "Dwgs.User") (width 0.15))
   (gr_line (start 391.4775 199.39) (end 396.5575 199.39) (layer "Dwgs.User") (width 0.15))
   (gr_line (start 396.5575 82.55) (end 396.5575 232.41) (layer "Dwgs.User") (width 0.15))
+  (gr_line (start 368.6175 232.41) (end 368.6175 191.77) (layer "Edge.Cuts") (width 0.1))
+  (gr_line (start 46.0375 127) (end 46.0375 232.41) (layer "Edge.Cuts") (width 0.1))
+  (gr_line (start 368.6175 191.77) (end 383.8575 191.77) (layer "Edge.Cuts") (width 0.1))
+  (gr_line (start 46.0375 127) (end 96.8375 127) (layer "Edge.Cuts") (width 0.1))
+  (gr_line (start 383.8575 95.25) (end 96.8375 95.25) (layer "Edge.Cuts") (width 0.1))
+  (gr_line (start 96.8375 127) (end 96.8375 95.25) (layer "Edge.Cuts") (width 0.1))
+  (gr_line (start 46.0375 232.41) (end 368.6175 232.41) (layer "Edge.Cuts") (width 0.1))
+  (gr_line (start 383.8575 191.77) (end 383.8575 95.25) (layer "Edge.Cuts") (width 0.1))
 )

Commit message: placing components
Parts:
- added C1: 100n, Capacitor_THT:C_Disc_D9.0mm_W2.5mm_P5.00mm, F.Cu at (142.6, 36.8)
- added C2: 100n, Capacitor_THT:C_Disc_D9.0mm_W2.5mm_P5.00mm, F.Cu at (126.7, 41.6)
- added C3: 100n, Capacitor_THT:C_Disc_D9.0mm_W2.5mm_P5.00mm, F.Cu at (137.3, 41.6)
- added C4: 22u, Capacitor_THT:CP_Radial_D5.0mm_P2.00mm, F.Cu at (147.4, 42.1)
- added D1: D, Diode_THT:D_DO-34_SOD68_P10.16mm_Horizontal, F.Cu at (75.2, 257.8)
- added D10: D, Diode_THT:D_DO-34_SOD68_P10.16mm_Horizontal, F.Cu at (310.2, 215.9)
- added D2: D, Diode_THT:D_DO-34_SOD68_P10.16mm_Horizontal, F.Cu at (85.4, 264.2)
- added D3: D, Diode_THT:D_DO-34_SOD68_P10.16mm_Horizontal, F.Cu at (328.0, 205.7)
- added D4: D, Diode_THT:D_DO-34_SOD68_P10.16mm_Horizontal, F.Cu at (325.4, 205.7)
- added D5: D, Diode_THT:D_DO-34_SOD68_P10.16mm_Horizontal, F.Cu at (322.9, 205.7)
- added D6: D, Diode_THT:D_DO-34_SOD68_P10.16mm_Horizontal, F.Cu at (320.4, 205.7)
- added D7: D, Diode_THT:D_DO-34_SOD68_P10.16mm_Horizontal, F.Cu at (317.8, 205.7)
- added D8: D, Diode_THT:D_DO-34_SOD68_P10.16mm_Horizontal, F.Cu at (315.3, 205.7)
- added D9: D, Diode_THT:D_DO-34_SOD68_P10.16mm_Horizontal, F.Cu at (312.7, 215.9)
- added IC1: 74LS161, Package_DIP:DIP-16_W7.62mm, F.Cu at (298.8, 106.7)
- added IC2: 74251, Package_DIP:DIP-16_W7.62mm, F.Cu at (136.2, 106.7)
- added IC3: 74145, Package_DIP:DIP-16_W7.62mm, F.Cu at (328.0, 106.7)
- added IC4: 74LS30, Package_DIP:DIP-14_W7.62mm, F.Cu at (357.2, 106.7)
- added PL1: Conn_01x17, Connector_PinHeader_2.54mm:PinHeader_1x17_P2.54mm_Horizontal, F.Cu at (161.6, 99.6)
- added R1: 470, Resistor_THT:R_Axial_DIN0309_L9.0mm_D3.2mm_P12.70mm_Horizontal, F.Cu at (125.5, 37.2)
- added R2: 470, Resistor_THT:R_Axial_DIN0309_L9.0mm_D3.2mm_P12.70mm_Horizontal, F.Cu at (141.4, 32.4)
- added R3: 470, Resistor_THT:R_Axial_DIN0309_L9.0mm_D3.2mm_P12.70mm_Horizontal, F.Cu at (125.5, 32.4)
- added SW74: SW_DIP_x08, Button_Switch_THT:SW_DIP_SPSTx08_Slide_9.78x22.5mm_W7.62mm_P2.54mm, F.Cu at (345.8, 219.7)

Commit message: start some routing
Parts:
- moved C3 247.3 mm to (377.5, 100.4), turned to -90 degrees
- moved C1 165.1 mm to (295.0, 100.4), turned to -90 degrees
- moved R2 74.1 mm to (118.4, 102.9), turned to 180 degrees
- moved R1 71.1 mm to (118.4, 108.0), turned to 180 degrees
- moved R3 65.7 mm to (118.4, 97.8), turned to 180 degrees
- moved C2 59.1 mm to (132.4, 100.4), turned to -90 degrees
- moved D10 10.2 mm to (310.2, 205.7), turned to -90 degrees
- moved D9 10.2 mm to (312.7, 205.7), turned to -90 degrees
Routing:
- net Net-(LD1-Pad1): track 0.00 -> 189.7 mm
- net Net-(LD2-Pad1): track 0.00 -> 181.8 mm
- net Net-(LD3-Pad1): track 0.00 -> 172.0 mm
- net Net-(D10-Pad2): track 0.00 -> 46.6 mm
- net Net-(D9-Pad2): track 0.00 -> 40.7 mm
- net Net-(D8-Pad2): track 0.00 -> 34.8 mm
- net Net-(D7-Pad2): track 0.00 -> 29.0 mm
- net Net-(D6-Pad2): track 0.00 -> 23.1 mm
- net Net-(D5-Pad2): track 0.00 -> 17.2 mm
- net Net-(D4-Pad2): track 0.00 -> 11.3 mm
- net Net-(D3-Pad2): track 0.00 -> 3.81 mm

Commit message: rotate switches 180 degrees
Parts:
- turned SW1 to 180 degrees
- turned SW10 to 180 degrees
- turned SW11 to 180 degrees
- turned SW12 to 180 degrees
- turned SW13 to 180 degrees
- turned SW14 to 180 degrees
- turned SW15 to 180 degrees
- turned SW16 to 180 degrees
- turned SW17 to 180 degrees
- turned SW18 to 180 degrees
- turned SW19 to 180 degrees
- turned SW2 to 180 degrees
- turned SW20 to 180 degrees
- turned SW21 to 180 degrees
- turned SW22 to 180 degrees
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
Commit message: start routing
Parts:
- moved RP1 131.6 mm to (349.6, 113.0)
- moved D2 64.8 mm to (122.2, 210.8), turned to 180 degrees
- moved D1 55.1 mm to (82.9, 203.2), turned to -90 degrees
- moved R1 5.08 mm to (118.4, 102.9)
- moved R2 5.08 mm to (118.4, 108.0)
- moved LD1 1.80 mm to (114.6, 223.5), turned to -90 degrees
- moved LD2 1.80 mm to (94.3, 223.5), turned to -90 degrees
- moved LD3 1.80 mm to (74.0, 223.5), turned to -90 degrees
Routing:
- net /Key Matrix/KC_ROW6: track 0.00 -> 531.7 mm
- net /Key Matrix/KC_ROW0: track 0.00 -> 494.1 mm
- net /Key Matrix/KC_COL2: track 0.00 -> 472.7 mm
- net /Key Matrix/KC_ROW3: track 0.00 -> 458.4 mm
- net /Key Matrix/KC_ROW4: track 0.00 -> 458.3 mm
- net /Key Matrix/KC_ROW5: track 0.00 -> 456.7 mm, vias 0 -> 1
- net /Key Matrix/KC_COL3: track 0.00 -> 453.8 mm
- net GND: track 0.00 -> 424.0 mm
- net /Key Matrix/KC_ROW7: track 0.00 -> 416.5 mm
- net /Key Matrix/KC_COL4: track 0.00 -> 391.7 mm
- net /Key Matrix/KC_ROW2: track 0.00 -> 384.2 mm
- net VCC: track 0.00 -> 384.1 mm
- net /Key Matrix/KC_COL0: track 0.00 -> 361.5 mm
- net /Key Matrix/KC_ROW1: track 0.00 -> 347.1 mm
- net /Key Matrix/KC_COL5: track 0.00 -> 345.4 mm
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
Commit message: routed rhs
Parts:
- moved RP1 34.2 mm to (375.0, 135.9), turned to 90 degrees
- moved C3 24.1 mm to (353.4, 100.4)
Connections:
- RP1 pad 3: /Key Matrix/KC_ROW1 -> /Key Matrix/KC_ROW6
- RP1 pad 4: /Key Matrix/KC_ROW2 -> /Key Matrix/KC_ROW5
- RP1 pad 5: /Key Matrix/KC_ROW3 -> /Key Matrix/KC_ROW4
- RP1 pad 6: /Key Matrix/KC_ROW4 -> /Key Matrix/KC_ROW3
- RP1 pad 7: /Key Matrix/KC_ROW5 -> /Key Matrix/KC_ROW2
- RP1 pad 8: /Key Matrix/KC_ROW6 -> /Key Matrix/KC_ROW1
Routing:
- net VCC: track 384.1 -> 592.0 mm
- net /CA2: track 0.00 -> 180.7 mm
- net /KB~{EN}: track 31.5 -> 179.0 mm
- net GND: track 424.0 -> 289.8 mm
- net /Key Matrix/KC_ROW4: track 458.3 -> 577.8 mm
- net /Key Matrix/KC_ROW3: track 458.4 -> 571.6 mm
- net /Key Matrix/KC_ROW1: track 347.1 -> 442.7 mm
- net /Key Matrix/KC_ROW2: track 384.2 -> 446.5 mm
- net /PA7: track 0.00 -> 45.2 mm, vias 0 -> 1
- net /Key Matrix/KC_ROW0: track 494.1 -> 464.3 mm
- net Net-(IC1-Pad11): track 4.47 -> 30.4 mm
- net /Key Matrix/KC_ROW7: track 416.5 -> 442.2 mm
- net /PA5: track 0.00 -> 25.4 mm
- net /PA6: track 0.00 -> 24.9 mm
- net /PA4: track 0.00 -> 24.5 mm
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
Commit message: tidy routing
Routing:
- net /Key Matrix/KC_ROW2: track 446.5 -> 428.6 mm
- net /Key Matrix/KC_ROW6: track 545.0 -> 530.5 mm
- net /Key Matrix/KC_ROW0: track 464.3 -> 451.5 mm
- net /Key Matrix/KC_ROW3: track 571.6 -> 559.9 mm
- net /Key Matrix/KC_ROW1: track 442.7 -> 435.2 mm
- net /Key Matrix/KC_ROW5: track 477.7 -> 471.4 mm
- net /Key Matrix/KC_ROW4: track 577.8 -> 571.9 mm
