File: KiCad/bbc-keyboard/bbc-keyboard.kicad_sch (KiCad schematic)
At the start: 31 parts

Commit message: FIX: mounting holes larger
Parts:
- H1, H2, H3, H4, H5, H6, H7, H8: footprint MountingHole:MountingHole_2.7mm_M2.5_DIN965_Pad -> MountingHole:MountingHole_3.2mm_M3_DIN965_Pad
Changed lines of the file:
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@@
     (property "Reference" "H1" (id 0) (at 42.545 139.065 90))
     (property "Value" "bkplt" (id 1) (at 33.655 140.335 90))
-    (property "Footprint" "MountingHole:MountingHole_2.7mm_M2.5_DIN965_Pad" (id 2) (at 40.005 140.335 0)
+    (property "Footprint" "MountingHole:MountingHole_3.2mm_M3_DIN965_Pad" (id 2) (at 40.005 140.335 0)
       (effects (font (size 1.27 1.27)) hide)
     )
@@
     (property "Reference" "H6" (id 0) (at 42.545 164.465 90))
     (property "Value" "bkplt" (id 1) (at 33.655 165.735 90))
-    (property "Footprint" "MountingHole:MountingHole_2.7mm_M2.5_DIN965_Pad" (id 2) (at 40.005 165.735 0)
+    (property "Footprint" "MountingHole:MountingHole_3.2mm_M3_DIN965_Pad" (id 2) (at 40.005 165.735 0)
       (effects (font (size 1.27 1.27)) hide)
     )
@@
     (property "Reference" "H2" (id 0) (at 42.545 144.145 90))
     (property "Value" "bkplt" (id 1) (at 33.655 145.415 90))
-    (property "Footprint" "MountingHole:MountingHole_2.7mm_M2.5_DIN965_Pad" (id 2) (at 40.005 145.415 0)
+    (property "Footprint" "MountingHole:MountingHole_3.2mm_M3_DIN965_Pad" (id 2) (at 40.005 145.415 0)
       (effects (font (size 1.27 1.27)) hide)
     )
@@
     (property "Reference" "H7" (id 0) (at 93.345 139.065 90))
     (property "Value" "front" (id 1) (at 84.455 140.335 90))
-    (property "Footprint" "MountingHole:MountingHole_2.7mm_M2.5_DIN965_Pad" (id 2) (at 90.805 140.335 0)
+    (property "Footprint" "MountingHole:MountingHole_3.2mm_M3_DIN965_Pad" (id 2) (at 90.805 140.335 0)
       (effects (font (size 1.27 1.27)) hide)
     )
@@
     (property "Reference" "H5" (id 0) (at 42.545 159.385 90))
     (property "Value" "bkplt" (id 1) (at 33.655 160.655 90))
-    (property "Footprint" "MountingHole:MountingHole_2.7mm_M2.5_DIN965_Pad" (id 2) (at 40.005 160.655 0)
+    (property "Footprint" "MountingHole:MountingHole_3.2mm_M3_DIN965_Pad" (id 2) (at 40.005 160.655 0)
       (effects (font (size 1.27 1.27)) hide)
     )
@@
     (property "Reference" "H8" (id 0) (at 93.345 144.145 90))
     (property "Value" "front" (id 1) (at 84.455 145.415 90))
-    (property "Footprint" "MountingHole:MountingHole_2.7mm_M2.5_DIN965_Pad" (id 2) (at 90.805 145.415 0)
+    (property "Footprint" "MountingHole:MountingHole_3.2mm_M3_DIN965_Pad" (id 2) (at 90.805 145.415 0)
       (effects (font (size 1.27 1.27)) hide)
     )
@@
     (property "Reference" "H4" (id 0) (at 42.545 154.305 90))
     (property "Value" "bkplt" (id 1) (at 33.655 155.575 90))
-    (property "Footprint" "MountingHole:MountingHole_2.7mm_M2.5_DIN965_Pad" (id 2) (at 40.005 155.575 0)
+    (property "Footprint" "MountingHole:MountingHole_3.2mm_M3_DIN965_Pad" (id 2) (at 40.005 155.575 0)
       (effects (font (size 1.27 1.27)) hide)
     )
@@
     (property "Reference" "H3" (id 0) (at 42.545 149.225 90))
     (property "Value" "bkplt" (id 1) (at 33.655 150.495 90))
-    (property "Footprint" "MountingHole:MountingHole_2.7mm_M2.5_DIN965_Pad" (id 2) (at 40.005 150.495 0)
+    (property "Footprint" "MountingHole:MountingHole_3.2mm_M3_DIN965_Pad" (id 2) (at 40.005 150.495 0)
       (effects (font (size 1.27 1.27)) hide)
     )
@@
     )
     (path "/106c5e61-c333-43ca-a561-c4ddf4ce6516"
-      (reference "H1") (unit 1) (value "bkplt") (footprint "MountingHole:MountingHole_2.7mm_M2.5_DIN965_Pad")
+      (reference "H1") (unit 1) (value "bkplt") (footprint "MountingHole:MountingHole_3.2mm_M3_DIN965_Pad")
     )
     (path "/5a832c11-9480-427b-bfda-2f6d86340ab6"
-      (reference "H2") (unit 1) (value "bkplt") (footprint "MountingHole:MountingHole_2.7mm_M2.5_DIN965_Pad")
+      (reference "H2") (unit 1) (value "bkplt") (footprint "MountingHole:MountingHole_3.2mm_M3_DIN965_Pad")
     )
     (path "/d0ca8ab4-7c56-4cc0-9a0f-c5b5ebf13e7e"
-      (reference "H3") (unit 1) (value "bkplt") (footprint "MountingHole:MountingHole_2.7mm_M2.5_DIN965_Pad")
+      (reference "H3") (unit 1) (value "bkplt") (footprint "MountingHole:MountingHole_3.2mm_M3_DIN965_Pad")
     )
     (path "/99505076-5b75-4ea0-9762-f32e1a7e1e76"
-      (reference "H4") (unit 1) (value "bkplt") (footprint "MountingHole:MountingHole_2.7mm_M2.5_DIN965_Pad")
+      (reference "H4") (unit 1) (value "bkplt") (footprint "MountingHole:MountingHole_3.2mm_M3_DIN965_Pad")
     )
     (path "/76b9f392-3aae-495d-b604-9c8647dadcc3"
-      (reference "H5") (unit 1) (value "bkplt") (footprint "MountingHole:MountingHole_2.7mm_M2.5_DIN965_Pad")
+      (reference "H5") (unit 1) (value "bkplt") (footprint "MountingHole:MountingHole_3.2mm_M3_DIN965_Pad")
     )
     (path "/207a956e-fa59-4412-ab85-b82d2c44089c"
-      (reference "H6") (unit 1) (value "bkplt") (footprint "MountingHole:MountingHole_2.7mm_M2.5_DIN965_Pad")
+      (reference "H6") (unit 1) (value "bkplt") (footprint "MountingHole:MountingHole_3.2mm_M3_DIN965_Pad")
     )
     (path "/723eb03a-f063-4883-8f37-23c6a99bfa03"
-      (reference "H7") (unit 1) (value "front") (footprint "MountingHole:MountingHole_2.7mm_M2.5_DIN965_Pad")
+      (reference "H7") (unit 1) (value "front") (footprint "MountingHole:MountingHole_3.2mm_M3_DIN965_Pad")
     )
     (path "/94b77a50-83e7-46ba-a832-3199d4958709"
-      (reference "H8") (unit 1) (value "front") (footprint "MountingHole:MountingHole_2.7mm_M2.5_DIN965_Pad")
+      (reference "H8") (unit 1) (value "front") (footprint "MountingHole:MountingHole_3.2mm_M3_DIN965_Pad")
     )
     (path "/89728ebf-3bac-4567-a498-e6be30f2bdc2"
