File: KiCad/model-b-ear-left/model-b-ear-left.kicad_sch (KiCad schematic)
At the start: 7 parts

Commit message: Ooops - didn't save, include correct mounting holes
Parts:
- H4, H5, H6: footprint Holes:SquareHole_6.5mm -> MountingHole:MountingHole_3.2mm_M3_DIN965
- H7: footprint Holes:SquareHole_6.5mm -> MountingHole:MountingHole_4.3mm_M4
Changed lines of the file:
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@@
       (effects (font (size 1.27 1.27)) (justify left))
     )
-    (property "Footprint" "Holes:SquareHole_6.5mm" (id 2) (at 102.87 58.42 0)
+    (property "Footprint" "MountingHole:MountingHole_3.2mm_M3_DIN965" (id 2) (at 102.87 58.42 0)
       (effects (font (size 1.27 1.27)) hide)
     )
@@
       (effects (font (size 1.27 1.27)) (justify left))
     )
-    (property "Footprint" "Holes:SquareHole_6.5mm" (id 2) (at 102.87 68.58 0)
+    (property "Footprint" "MountingHole:MountingHole_3.2mm_M3_DIN965" (id 2) (at 102.87 68.58 0)
       (effects (font (size 1.27 1.27)) hide)
     )
@@
       (effects (font (size 1.27 1.27)) (justify left))
     )
-    (property "Footprint" "Holes:SquareHole_6.5mm" (id 2) (at 102.87 73.66 0)
+    (property "Footprint" "MountingHole:MountingHole_4.3mm_M4" (id 2) (at 102.87 73.66 0)
       (effects (font (size 1.27 1.27)) hide)
     )
@@
       (effects (font (size 1.27 1.27)) (justify left))
     )
-    (property "Footprint" "Holes:SquareHole_6.5mm" (id 2) (at 102.87 63.5 0)
+    (property "Footprint" "MountingHole:MountingHole_3.2mm_M3_DIN965" (id 2) (at 102.87 63.5 0)
       (effects (font (size 1.27 1.27)) hide)
     )
@@
     )
     (path "/1b843358-5065-483e-81b3-fd95d08fc9f3"
-      (reference "H4") (unit 1) (value "HoleThru") (footprint "Holes:SquareHole_6.5mm")
+      (reference "H4") (unit 1) (value "HoleThru") (footprint "MountingHole:MountingHole_3.2mm_M3_DIN965")
     )
     (path "/f1a89646-ce1e-4644-8c9f-82a8e916245f"
-      (reference "H5") (unit 1) (value "HoleThru") (footprint "Holes:SquareHole_6.5mm")
+      (reference "H5") (unit 1) (value "HoleThru") (footprint "MountingHole:MountingHole_3.2mm_M3_DIN965")
     )
     (path "/28ce1be0-6097-46dd-8885-62587b78d840"
-      (reference "H6") (unit 1) (value "HoleThru") (footprint "Holes:SquareHole_6.5mm")
+      (reference "H6") (unit 1) (value "HoleThru") (footprint "MountingHole:MountingHole_3.2mm_M3_DIN965")
     )
     (path "/a2851980-f2f3-42ee-b3b4-6e46ec2b5341"
-      (reference "H7") (unit 1) (value "HoleThru") (footprint "Holes:SquareHole_6.5mm")
+      (reference "H7") (unit 1) (value "HoleThru") (footprint "MountingHole:MountingHole_4.3mm_M4")
     )
   )
